File: kicad/pcb/ATmega32_USART_Serial_Data_Monitor_System_v001.kicad_pcb (KiCad board)
At the start: 2 copper layers, 107.5 x 100.5 mm, 15 parts, among them J1 Conn_01x04, SW1 SW_Push, SW2 SW_Push, SW3 SW_Push, U1 ATmega32A, Y1 8MHz

Commit message: Add files via upload
Parts:
- added DS1: WC1602A, Display:WC1602A, F.Cu at (163.6, 80.5)
- added RV1: R_Potentiometer, Potentiometer_THT:Potentiometer_Bourns_3296W_Vertical, F.Cu at (168.5, 145.0)
- moved D1 45.6 mm to (205.5, 104.0)
- moved D2 45.6 mm to (204.5, 95.5)
- moved R1 45.6 mm to (188.8, 103.0)
- moved R2 45.6 mm to (188.8, 93.0)
- moved C4 22.6 mm to (111.0, 153.0)
- moved C3 22.6 mm to (111.0, 145.5)
- moved R3 22.6 mm to (103.8, 140.0)
- moved SW1 22.6 mm to (89.7, 96.2)
- moved SW2 22.6 mm to (98.2, 96.2)
- moved Y1 22.6 mm to (128.9, 142.5)
- moved SW3 22.6 mm to (106.8, 96.2)
- moved U1 22.6 mm to (98.0, 132.2)
- moved C1 22.6 mm to (142.5, 145.5)
- moved C2 22.6 mm to (142.5, 138.5)
- moved J1 21.3 mm to (159.4, 108.0)
Connections:
- D1 pad 1: Net-(D1-K) -> GND
- D1 pad 2: GND -> Net-(D1-A)
- R1 pad 2: Net-(D1-K) -> Net-(D1-A)
- U1 pad 22: unconnected-(U1-PC0-Pad22) -> Net-(DS1-RS)
- U1 pad 23: unconnected-(U1-PC1-Pad23) -> Net-(DS1-E)
- U1 pad 24: unconnected-(U1-PC2-Pad24) -> Net-(DS1-D4)
- U1 pad 25: unconnected-(U1-PC3-Pad25) -> Net-(DS1-D5)
- U1 pad 26: unconnected-(U1-PC4-Pad26) -> Net-(DS1-D6)
- U1 pad 27: unconnected-(U1-PC5-Pad27) -> Net-(DS1-D7)
Routing:
- net VCC: track 65.6 -> 226.5 mm
- net GND: track 181.6 -> 336.1 mm
- net Net-(U1-PB1): track 56.3 -> 145.2 mm
- net Net-(DS1-VO): track 0.00 -> 67.6 mm
- net Net-(DS1-RS): track 0.00 -> 41.5 mm
- net Net-(DS1-E): track 0.00 -> 40.5 mm
- net Net-(DS1-D5): track 0.00 -> 36.7 mm
- net Net-(DS1-D7): track 0.00 -> 36.7 mm
- net Net-(DS1-D6): track 0.00 -> 36.7 mm
- net Net-(DS1-D4): track 0.00 -> 36.7 mm
- net Net-(D1-K): track 32.0 -> 0.00 mm
- net Net-(D1-A): track 0.00 -> 24.9 mm
- net Net-(U1-PB2): track 111.5 -> 131.3 mm
- net Net-(J1-Pin_3): track 26.4 -> 40.9 mm
- net Net-(J1-Pin_2): track 26.4 -> 40.9 mm
Other:
- board size 107.5 x 100.5 mm -> 166.5 x 129.5 mm
