File: kicad/schematic/ATmega32_USART_Serial_Data_Monitor_System_v001.kicad_sch (KiCad schematic)
At the start: 17 parts, among them J1 Conn_01x04, SW1 SW_Push, SW2 SW_Push, SW3 SW_Push, SW4 SW_Push, SW5 SW_Push, U1 ATmega32A-P, Y1 8MHz

Commit message: Add files via upload
Parts:
- removed SW4, SW5: SW_Push, Button_Switch_THT:SW_PUSH_6mm, symbol Switch:SW_Push
- C3, C4: value 100nF -> 100pF
- U1: value ATmega32A-P -> ATmega32A
Connections:
- net GND: now also D1.1 (K); no longer D1.2 (A)
- net at R1.2: now also D1.2 (A); no longer D1.1 (K)

Commit message: Add files via upload
Parts:
- added DS1: WC1602A, Display:WC1602A, symbol Display_Character:WC1602A
- added RV1: R_Potentiometer, Potentiometer_THT:Potentiometer_Bourns_3296W_Vertical, symbol Device:R_Potentiometer
Connections:
- net GND: now also DS1.1 (VSS), DS1.16 (LED(-)), DS1.5 (R/W), RV1.3
- net VCC: now also DS1.15 (LED(+)), DS1.2 (VDD), RV1.1
- net at U1.22 (PC0): now also DS1.4 (RS)
- net at U1.23 (PC1): now also DS1.6 (E)
- net at U1.24 (PC2): now also DS1.11 (D4)
- net at U1.25 (PC3): now also DS1.12 (D5)
- net at U1.26 (PC4): now also DS1.13 (D6)
- net at U1.27 (PC5): now also DS1.14 (D7)
- new net: DS1.3 (VO), RV1.2
- no-connect marks 26 -> 24
